Commit message: add real time planner

File: robot_description/urdf/ur10.urdf.xacro (robot description, xacro)
@@ -61,5 +61,5 @@
       <mass
         value="50.0" />
-      <inertia ixx="1.0" ixy="0.0" ixz="0.0" iyy="1.0" iyz="0.0" izz="1.0" />
+      <inertia ixx="50.0" ixy="0.0" ixz="0.0" iyy="50.0" iyz="0.0" izz="50.0" />
     </inertial>
     <visual>
